File: Xenia-1-rocket-schematic.sch/Xenia-1-rocket-schematic.sch.kicad_sch (KiCad schematic)
At the start: 33 parts, among them M1 Stepper_Motor_bipolar, U3 A1115, U6 BME280, U7 Black_Box

Commit message: Updated the schematic
Labeled the sides of the avionics bay and wired the buzzer to the DIR pin
Connections:
- net +5V: no longer U?. (PWR)
- net 5V: no longer U?. (PWR)
- net GPIO27/DIR: now also U?. (PWR)
- net GPIO7: now also U?. (PWR)
- net at U?.~ (V_in): now also BT?.2 (-)
Other:
- note added: "Bottom of the Command Module"
- note added: "Side A"
- note added: "Side B"
- note added: "Side C"
- note added: "Side D"
- note added: "Top of Command Module"
- moved on the sheet: U?
Changed lines of the file:
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@@
   (junction (at 331.47 276.86) (diameter 0) (color 0 0 0 0)
   )
+  (junction (at 375.92 134.62) (diameter 0) (color 0 0 0 0)
+  )
   (junction (at 420.37 224.79) (diameter 0) (color 0 0 0 0)
   )
@@
   )
   (junction (at 83.82 19.05) (diameter 0) (color 0 0 0 0)
-  )
-  (junction (at 389.89 134.62) (diameter 0) (color 0 0 0 0)
   )
   (junction (at 341.63 236.22) (diameter 0) (color 0 0 0 0)
@@
     (stroke (width 0) (type default) (color 0 0 0 0))
   )
+  (wire (pts (xy 375.92 134.62) (xy 439.42 134.62))
+    (stroke (width 0) (type default) (color 0 0 0 0))
+  )
   (wire (pts (xy 308.61 63.5) (xy 326.39 63.5))
     (stroke (width 0) (type default) (color 0 0 0 0))
@@
     (stroke (width 0) (type default) (color 0 0 0 0))
   )
+  (wire (pts (xy 375.92 134.62) (xy 375.92 88.9))
+    (stroke (width 0) (type default) (color 0 0 0 0))
+  )
   (polyline (pts (xy 579.12 116.84) (xy 581.66 116.84))
     (stroke (width 0) (type default) (color 0 0 0 0))
@@
     (stroke (width 0) (type default) (color 0 0 0 0))
   )
-  (wire (pts (xy 375.92 147.32) (xy 375.92 88.9))
+  (wire (pts (xy 375.92 147.32) (xy 375.92 134.62))
     (stroke (width 0) (type default) (color 0 0 0 0))
   )
@@
     (stroke (width 0) (type default) (color 0 0 0 0))
   )
-  (wire (pts (xy 389.89 134.62) (xy 389.89 153.67))
-    (stroke (width 0) (type default) (color 0 0 0 0))
-  )
   (wire (pts (xy 386.08 127) (xy 541.02 127))
     (stroke (width 0) (type default) (color 0 0 0 0))
@@
     (stroke (width 0) (type default) (color 0 0 0 0))
   )
-  (wire (pts (xy 389.89 58.42) (xy 389.89 134.62))
+  (wire (pts (xy 389.89 58.42) (xy 389.89 153.67))
     (stroke (width 0) (type default) (color 0 0 0 0))
   )
@@
     (stroke (width 0) (type default) (color 0 0 0 0))
   )
-  (wire (pts (xy 439.42 134.62) (xy 389.89 134.62))
-    (stroke (width 0) (type default) (color 0 0 0 0))
-  )
   (wire (pts (xy 346.71 236.22) (xy 341.63 236.22))
     (stroke (width 0) (type default) (color 0 0 0 0))
@@
   (wire (pts (xy 337.82 151.13) (xy 378.46 151.13))
     (stroke (width 0) (type default) (color 0 0 0 0))
+  )
+  (text "Side B" (at 491.49 71.12 0)
+    (effects (font (size 3 3)) (justify left bottom))
   )
   (text "IMU" (at 199.39 132.08 0)
     (effects (font (size 1.27 1.27)) (justify left bottom))
   )
+  (text "Side C" (at 553.72 127 0)
+    (effects (font (size 3 3)) (justify left bottom))
+  )
+  (text "Top of Command Module" (at 490.22 27.94 0)
+    (effects (font (size 3 3)) (justify left bottom))
+  )
+  (text "Side D" (at 524.51 209.55 0)
+    (effects (font (size 3 3)) (justify left bottom))
+  )
+  (text "Side A" (at 543.56 294.64 0)
+    (effects (font (size 3 3)) (justify left bottom))
+  )
   (text "Pi" (at 19.05 124.46 0)
     (effects (font (size 1.27 1.27)) (justify left bottom))
   )
   (text "Inputs" (at 161.29 58.42 0)
-    (effects (font (size 1.27 1.27)) (justify left bottom))
+    (effects (font (size 4 4)) (justify left bottom))
   )
   (text "I2C Sensors" (at 139.7 125.73 0)
-    (effects (font (size 1.27 1.27)) (justify left bottom))
-  )
-  (text "Outputs" (at 93.98 81.28 0)
-    (effects (font (size 1.27 1.27)) (justify left bottom))
+    (effects (font (size 4 4)) (justify left bottom))
+  )
+  (text "Outputs" (at 62.23 78.74 0)
+    (effects (font (size 4 4)) (justify left bottom))
+  )
+  (text "Bottom of \nthe\nCommand\nModule" (at 270.51 297.18 0)
+    (effects (font (size 3 3)) (justify left bottom))
   )
   (text "Barometric Pressure Sensor" (at 243.84 191.77 0)
@@
   )
   (label "GPIO9" (at 251.46 24.13 180)
+    (effects (font (size 1.27 1.27)) (justify right bottom))
+  )
+  (label "GPIO7" (at 97.79 109.22 180)
     (effects (font (size 1.27 1.27)) (justify right bottom))
   )
@@
     (pin "~")
   )
-  (symbol (lib_id "Rocketry_project:Strain Gauge PCB") (at 349.25 337.82 270) (unit 1)
-    (in_bom yes) (on_board yes) (fields_autoplaced)
-    (property "Reference" "U?" (id 0) (at 353.7712 363.6553 90)
-      (effects (font (size 1.27 1.27)) (justify left))
-    )
-    (property "Value" "Strain Gauge PCB" (id 1) (at 353.7712 366.1922 90)
-      (effects (font (size 1.27 1.27)) (justify left))
-    )
-    (property "Footprint" "" (id 2) (at 349.25 337.82 0)
-      (effects (font (size 1.27 1.27)) hide)
-    )
-    (property "Datasheet" "" (id 3) (at 349.25 337.82 0)
+  (symbol (lib_id "Rocketry_project:Strain Gauge PCB") (at 284.48 330.2 270) (unit 1)
+    (in_bom yes) (on_board yes) (fields_autoplaced)
+    (property "Reference" "U?" (id 0) (at 289.0012 356.0353 90)
+      (effects (font (size 1.27 1.27)) (justify left))
+    )
+    (property "Value" "Strain Gauge PCB" (id 1) (at 289.0012 358.5722 90)
+      (effects (font (size 1.27 1.27)) (justify left))
+    )
+    (property "Footprint" "" (id 2) (at 284.48 330.2 0)
+      (effects (font (size 1.27 1.27)) hide)
+    )
+    (property "Datasheet" "" (id 3) (at 284.48 330.2 0)
       (effects (font (size 1.27 1.27)) hide)
     )
@@
     )
     (pin "~")
-  )
-  (symbol (lib_id "power:+5V") (at 97.79 109.22 0) (unit 1)
-    (in_bom yes) (on_board yes) (fields_autoplaced)
-    (property "Reference" "#PWR?" (id 0) (at 97.79 113.03 0)
-      (effects (font (size 1.27 1.27)) hide)
-    )
-    (property "Value" "+5V" (id 1) (at 97.79 105.6442 0))
-    (property "Footprint" "" (id 2) (at 97.79 109.22 0)
-      (effects (font (size 1.27 1.27)) hide)
-    )
-    (property "Datasheet" "" (id 3) (at 97.79 109.22 0)
-      (effects (font (size 1.27 1.27)) hide)
-    )
-    (pin "1")
   )
   (symbol (lib_name "LSM9DS1_1") (lib_id "Rocketry_project:LSM9DS1") (at 190.5 171.45 0) (unit 1)
@@
       (reference "#PWR?") (unit 1) (value "GND") (footprint "")
     )
-    (path "/3d373373-7625-4aa8-93b7-d71105c477a1"
-      (reference "#PWR?") (unit 1) (value "+5V") (footprint "")
-    )
     (path "/51c94b1c-75ed-430f-a70b-fe26d3a87f12"
