File: Xenia-1-rocket-schematic.sch/Xenia-1-rocket-schematic.sch.kicad_sch (KiCad schematic)
At the start: 65 parts, among them M1 Stepper_Motor_bipolar, M2 Stepper_Motor_bipolar, U1 E-Match, U10 Transmitter, U11 E-Match, U12 E-Match, U13 ADXL375, U14 Raven4, U15 LSM9DS1, U16 Strain Gauge PCB, U17 Strain Gauge PCB, U18 DRV8825, U19 BME280, U2 E-Match, U20 Black_Box, U21 A1115, U22 Buzzer, U23 LSM9DS1, U24 E-Match, U25 Camera, U26 ADXL375, U27 E-Match, U28 Raven4, U29 Raven4, U3 A1115, U30 E-Match, U31 Transmitter, U32 E-Match, U4 DRV8825, U5 Camera, U6 BME280, U7 Black_Box, U8 Raven4, U9 Buzzer

Commit message: Updated schematic
Moved two sensors around. Should be final version
Parts:
- removed U?: ADXL375, symbol Rocketry_project:ADXL375
- removed U?: BME280, symbol Rocketry_project:BME280
- added U?: ADXL375, symbol Rocketry_project:ADXL375
- added U?: BME280, symbol Rocketry_project:BME280
Connections:
- net 3V3: now also U?. (V_in), U?.~ (V_in)
- net GND: now also U?. (V_in), U?.~ (V_in)
- net I2C Clock: now also U?. (V_in), U?.~ (V_in)
- net I2C Data: now also U?. (V_in), U?.~ (V_in)
Changed lines of the file:
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@@
   (no_connect (at 201.93 170.18))
   (no_connect (at 201.93 173.99))
-  (no_connect (at 932.18 111.76))
-  (no_connect (at 932.18 107.95))
-  (no_connect (at 932.18 104.14))
-  (no_connect (at 932.18 100.33))
-  (no_connect (at 932.18 96.52))
-  (no_connect (at 908.05 96.52))
+  (no_connect (at 1005.84 330.2))
+  (no_connect (at 1005.84 337.82))
+  (no_connect (at 816.61 95.25))
+  (no_connect (at 816.61 110.49))
   (no_connect (at 908.05 111.76))
-  (no_connect (at 908.05 115.57))
-  (no_connect (at 908.05 119.38))
   (no_connect (at 908.05 123.19))
-  (no_connect (at 816.61 114.3))
-  (no_connect (at 816.61 106.68))
-  (no_connect (at 816.61 95.25))
+  (no_connect (at 908.05 119.38))
+  (no_connect (at 908.05 115.57))
+  (no_connect (at 908.05 96.52))
+  (no_connect (at 932.18 96.52))
+  (no_connect (at 932.18 107.95))
+  (no_connect (at 932.18 111.76))
+  (no_connect (at 932.18 100.33))
+  (no_connect (at 932.18 104.14))
   (no_connect (at 146.05 158.75))
   (no_connect (at 146.05 143.51))
@@
   (no_connect (at 495.3 208.28))
   (no_connect (at 495.3 212.09))
-  (no_connect (at 873.76 149.86))
   (no_connect (at 873.76 152.4))
-  (no_connect (at 873.76 162.56))
-  (no_connect (at 828.04 180.34))
+  (no_connect (at 873.76 149.86))
   (no_connect (at 828.04 177.8))
-  (no_connect (at 828.04 167.64))
+  (no_connect (at 873.76 180.34))
   (no_connect (at 873.76 170.18))
-  (no_connect (at 828.04 195.58))
+  (no_connect (at 828.04 180.34))
   (no_connect (at 873.76 182.88))
-  (no_connect (at 873.76 180.34))
+  (no_connect (at 828.04 195.58))
+  (no_connect (at 828.04 167.64))
+  (no_connect (at 873.76 162.56))
   (no_connect (at 227.33 146.05))
   (no_connect (at 227.33 149.86))
@@
   (no_connect (at 227.33 196.85))
   (no_connect (at 227.33 177.8))
+  (no_connect (at 960.12 331.47))
+  (no_connect (at 960.12 327.66))
+  (no_connect (at 974.09 241.3))
+  (no_connect (at 974.09 245.11))
+  (no_connect (at 974.09 248.92))
   (no_connect (at 1032.51 114.3))
   (no_connect (at 1032.51 118.11))
+  (no_connect (at 960.12 339.09))
   (no_connect (at 1040.13 250.19))
   (no_connect (at 1040.13 254))
-  (no_connect (at 960.12 331.47))
-  (no_connect (at 960.12 339.09))
   (no_connect (at 960.12 342.9))
-  (no_connect (at 960.12 327.66))
-  (no_connect (at 974.09 248.92))
-  (no_connect (at 974.09 245.11))
-  (no_connect (at 974.09 241.3))
-  (no_connect (at 960.12 346.71))
-  (no_connect (at 1005.84 334.01))
   (no_connect (at 1005.84 318.77))
-  (no_connect (at 1023.62 316.23))
-  (no_connect (at 1023.62 320.04))
-  (no_connect (at 1023.62 323.85))
-  (no_connect (at 1023.62 327.66))
+  (no_connect (at 960.12 346.71))
+  (no_connect (at 834.39 104.14))
+  (no_connect (at 834.39 100.33))
+  (no_connect (at 834.39 96.52))
+  (no_connect (at 834.39 92.71))
   (no_connect (at 77.47 165.1))
   (no_connect (at 77.47 167.64))
@@
     (stroke (width 0) (type default) (color 0 0 0 0))
   )
-  (wire (pts (xy 1005.84 330.2) (xy 975.36 330.2))
-    (stroke (width 0) (type default) (color 0 0 0 0))
-  )
   (wire (pts (xy 386.08 68.58) (xy 386.08 127))
     (stroke (width 0) (type default) (color 0 0 0 0))
@@
     (stroke (width 0) (type default) (color 0 0 0 0))
   )
+  (wire (pts (xy 816.61 106.68) (xy 815.34 106.68))
+    (stroke (width 0) (type default) (color 0 0 0 0))
+  )
   (wire (pts (xy 99.06 31.75) (xy 68.58 31.75))
     (stroke (width 0) (type default) (color 0 0 0 0))
@@
     (stroke (width 0) (type default) (color 0 0 0 0))
   )
-  (wire (pts (xy 816.61 110.49) (xy 815.34 110.49))
-    (stroke (width 0) (type default) (color 0 0 0 0))
-  )
   (wire (pts (xy 504.19 300.99) (xy 504.19 237.49))
     (stroke (width 0) (type default) (color 0 0 0 0))
@@
     (stroke (width 0) (type default) (color 0 0 0 0))
   )
+  (wire (pts (xy 1005.84 334.01) (xy 975.36 334.01))
+    (stroke (width 0) (type default) (color 0 0 0 0))
+  )
   (wire (pts (xy 808.99 91.44) (xy 816.61 91.44))
     (stroke (width 0) (type default) (color 0 0 0 0))
@@
     (stroke (width 0) (type default) (color 0 0 0 0))
   )
-  (wire (pts (xy 975.36 330.2) (xy 975.36 300.99))
+  (wire (pts (xy 975.36 300.99) (xy 975.36 334.01))
     (stroke (width 0) (type default) (color 0 0 0 0))
   )
@@
     (stroke (width 0) (type default) (color 0 0 0 0))
   )
-  (wire (pts (xy 815.34 110.49) (xy 815.34 124.46))
+  (wire (pts (xy 815.34 106.68) (xy 815.34 124.46))
     (stroke (width 0) (type default) (color 0 0 0 0))
   )
@@
     (pin "1")
   )
-  (symbol (lib_id "Rocketry_project:ADXL375") (at 1013.46 322.58 0) (unit 1)
+  (symbol (lib_id "Rocketry_project:ADXL375") (at 824.23 99.06 0) (unit 1)
     (in_bom yes) (on_board yes) (fields_autoplaced)
-    (property "Reference" "U?" (id 0) (at 1014.73 309.406 0))
-    (property "Value" "ADXL375" (id 1) (at 1014.73 311.9429 0))
-    (property "Footprint" "" (id 2) (at 1013.46 322.58 0)
+    (property "Reference" "U?" (id 0) (at 825.5 85.886 0))
+    (property "Value" "ADXL375" (id 1) (at 825.5 88.4229 0))
+    (property "Footprint" "" (id 2) (at 824.23 99.06 0)
       (effects (font (size 1.27 1.27)) hide)
     )
-    (property "Datasheet" "" (id 3) (at 1013.46 322.58 0)
+    (property "Datasheet" "" (id 3) (at 824.23 99.06 0)
       (effects (font (size 1.27 1.27)) hide)
     )
@@
     (pin "1")
   )
+  (symbol (lib_name "BME280_1") (lib_id "Rocketry_project:BME280") (at 1016 322.58 270) (unit 1)
+    (in_bom yes) (on_board yes)
+    (property "Reference" "U?" (id 0) (at 1023.62 326.39 90)
+      (effects (font (size 1.27 1.27)) (justify left))
+    )
+    (property "Value" "BME280" (id 1) (at 1021.715 330.6322 90)
+      (effects (font (size 1.27 1.27)) (justify left))
+    )
+    (property "Footprint" "" (id 2) (at 1016 322.58 0)
+      (effects (font (size 1.27 1.27)) hide)
+    )
+    (property "Datasheet" "" (id 3) (at 1016 322.58 0)
+      (effects (font (size 1.27 1.27)) hide)
+    )
+    (pin "~")
+    (pin "~")
+    (pin "~")
+    (pin "~")
+    (pin "~")
+    (pin "~")
+    (pin "~")
+  )
   (symbol (lib_id "power:GND") (at 111.76 78.74 0) (unit 1)
     (in_bom yes) (on_board yes) (fields_autoplaced)
@@
     (pin "1")
   )
-  (symbol (lib_name "BME280_1") (lib_id "Rocketry_project:BME280") (at 826.77 99.06 270) (unit 1)
-    (in_bom yes) (on_board yes) (fields_autoplaced)
-    (property "Reference" "U?" (id 0) (at 832.485 104.5753 90)
-      (effects (font (size 1.27 1.27)) (justify left))
-    )
-    (property "Value" "BME280" (id 1) (at 832.485 107.1122 90)
-      (effects (font (size 1.27 1.27)) (justify left))
-    )
-    (property "Footprint" "" (id 2) (at 826.77 99.06 0)
-      (effects (font (size 1.27 1.27)) hide)
-    )
-    (property "Datasheet" "" (id 3) (at 826.77 99.06 0)
-      (effects (font (size 1.27 1.27)) hide)
-    )
-    (pin "~")
-    (pin "~")
-    (pin "~")
-    (pin "~")
-    (pin "~")
-    (pin "~")
-    (pin "~")
-  )
   (symbol (lib_id "Motor:Stepper_Motor_bipolar") (at 92.71 44.45 0) (unit 1)
     (in_bom yes) (on_board yes) (fields_autoplaced)
@@
       (reference "U?") (unit 1) (value "LSM9DS1") (footprint "")
     )
-    (path "/9c6f7b0e-b236-4413-8f10-7b52613aea1d"
+    (path "/9f3d7f2e-abff-4c83-a34e-3e3d809d8c05"
       (reference "U?") (unit 1) (value "ADXL375") (footprint "")
     )
@@
       (reference "U?") (unit 1) (value "E-Match") (footprint "")
     )
+    (path "/b870f872-42dc-4210-800b-899d36550add"
+      (reference "U?") (unit 1) (value "BME280") (footprint "")
+    )
     (path "/be49d7d8-fbbb-491c-9f79-289e726cd71e"
       (reference "U?") (unit 1) (value "A1115") (footprint "")
@@
       (reference "U?") (unit 1) (value "E-Match") (footprint "")
     )
-    (path "/fd2798da-749d-4b27-a179-6a46f6db969e"
-      (reference "U?") (unit 1) (value "BME280") (footprint "")
-    )
   )

Commit message: Updated schematic
Made the schematic line up with the actual avionics bay
Parts:
- removed RV?: R_Potentiometer, symbol Device:R_Potentiometer
- removed U?: Buzzer, symbol Rocketry_project:Buzzer
- removed U?: Transmitter, symbol Rocketry_project:Transmitter
- removed U?: BME280, symbol Rocketry_project:BME280
- removed U?: A1115, symbol Rocketry_project:A1115
- added RV?: R_Potentiometer, symbol Device:R_Potentiometer
- added U?: A1115, symbol Rocketry_project:A1115
- added U?: Transmitter, symbol Rocketry_project:Transmitter
- added U?: Buzzer, symbol Rocketry_project:Buzzer
- added U?: BME280, symbol Rocketry_project:BME280
Connections:
- net TTL-DIN is gone; now on net 3V3: A1.8 (TXD0/GPIO14), A?.8 (TXD0/GPIO14)
- net 3V3: now also A2.3 (GPIO2/SDA), A?.3 (GPIO2/SDA), U21. (VDD), U?. (TTL-DOUT), U?. (VDD), U?.~ (V_in)
- net 5V: now also RV?.1, U?. (VDD)
- net DIR: now also U?. (PWR)
- net GND: now also RV?.3, U?. (PWR), U?. (TTL-DOUT), U?. (VDD), U?.~ (V_in)
- net I2C Clock: now also U?. (VDD), U?.~ (V_in)
- net TTL-DOUT: now also U?. (TTL-DOUT)
- removed net I2C Data: A2.3 (GPIO2/SDA), A?.3 (GPIO2/SDA), U19.~ (V_in), U21. (VDD), U23.~ (V_in), U26. (V_in), U?. (V_in), U?.~ (V_in)
- new net: RV?.2, U?. (VDD)
- no-connect marks 115 -> 112

Commit message: Updated schematic
Deleted old version of wiring side
Parts:
- removed A2: rPi0w2, ADA3708_RPI-ZERO, symbol ADA3708:rPi0w2
- removed BT2, BT3: Battery_Cell, symbol Device:Battery_Cell
- removed C2: CAP, symbol pspice:CAP
- removed M2: Stepper_Motor_bipolar, symbol Motor:Stepper_Motor_bipolar
- removed RV2: R_Potentiometer, symbol Device:R_Potentiometer
- removed U17: Strain Gauge PCB, symbol Rocketry_project:Strain Gauge PCB
- removed U18: DRV8825, symbol Rocketry_project:DRV8825
- removed U19: BME280, symbol Rocketry_project:BME280
- removed U20: Black_Box, symbol Rocketry_project:Black_Box
- removed U21: A1115, symbol Rocketry_project:A1115
- removed U22: Buzzer, symbol Rocketry_project:Buzzer
- removed U23: LSM9DS1, symbol Rocketry_project:LSM9DS1
- removed U24, U27, U30, U32: E-Match, symbol Rocketry_project:E-Match
- removed U25: Camera, symbol Rocketry_project:Camera
- removed U26: ADXL375, symbol Rocketry_project:ADXL375
- removed U28, U29: Raven4, symbol Rocketry_project:Raven4
- removed U31: Transmitter, symbol Rocketry_project:Transmitter
Connections:
- net I2C Clock is gone; now on net SCL: A?.5 (GPIO3/SCL), U?. (VDD), U?. (V_in), U?.~ (V_in), U?.~ (V_in)
- net APO: no longer U1. (Input), U?. (Input), U?. (Input)
- net SCL: now reaches U?. (VDD)
- net Main: now reaches U?.~ (V_in)
- net Main: now also U1. (Input), U?. (Input), U?. (Input), U?.~ (V_in)
- no-connect marks 112 -> 81
Other:
- note removed: "Bottom of the Command Module"
- note removed: "Top of Command Module"
